Commit message: Add wrist joint and curved gripper to SCARA
Expand the SCARA arm xacro to add a continuous wrist (J_wrist) and NEMA17 motor visuals, converting the model from a 4-DOF to a 5-DOF layout. Introduces new properties (wrist_motor, wrist_len, finger_r) and a darker material, adjusts inertial/visual sizes for link2, wrist and gripper base, and repositions the gripper mount to the wrist. Replaces the previous simple finger boxes with a curved_finger macro that creates two curved gripping fingers (left/right) using composed boxes, and keeps the prismatic grip joints but updates origins/limits/axes accordingly. All changes are contained in ros2_ws/src/arm_description/urdf/arm.xacro.

File: ros2_ws/src/arm_description/urdf/arm.xacro (robot description, xacro)
@@ -2,5 +2,7 @@
 <!-- =========================================================================
      arm.xacro
-     Tay robot SCARA (4 DOF): J1 vai + J2 khuyu + Z nang/ha + gripper kep.
+     Tay robot SCARA (5 DOF): J1 vai + J2 khuyu + Z nang/ha
+     + J_wrist xoay co tay 360 do (motor NEMA17 o dau canh tay 2)
+     + gripper kep 2 ngam cong om vat (mo/khep).
      Don vi: met, kg, rad. Macro doc lap, parent gan tuy y.
      ========================================================================= -->
@@ -13,7 +15,11 @@
   <xacro:property name="z_travel"     value="0.40"/>
   <xacro:property name="arm_mass"     value="0.5"/>
-  <xacro:property name="grip_open"    value="0.20"/>
-  <xacro:property name="finger_len"   value="0.06"/>
-  <xacro:property name="finger_thick" value="0.02"/>
+  <!-- co tay = motor NEMA17 chia xuong + cum trang xoay theo -->
+  <xacro:property name="wrist_motor"  value="0.042"/>  <!-- NEMA17 ~42mm -->
+  <xacro:property name="wrist_len"    value="0.07"/>   <!-- cao cum co tay (motor+de) -->
+  <!-- gripper: 2 ngam cong om vat tron -->
+  <xacro:property name="grip_open"    value="0.20"/>   <!-- mo toi da ~20cm -->
+  <xacro:property name="finger_r"     value="0.05"/>   <!-- ban kinh cung ngam -->
+  <xacro:property name="finger_thick" value="0.015"/>
   <xacro:macro name="arm_box_inertia" params="m x y z">
     <inertial>
@@ -26,4 +32,5 @@
   <material name="arm_blue"><color rgba="0.15 0.35 0.85 1.0"/></material>
   <material name="arm_white"><color rgba="0.95 0.95 0.95 1.0"/></material>
+  <material name="arm_dark"><color rgba="0.15 0.15 0.18 1.0"/></material>
   <xacro:macro name="scara_arm" params="parent xyz:='0 0 0' rpy:='0 0 0'">
     <link name="arm_base_link">
@@ -80,4 +87,10 @@
         <material name="arm_blue"/>
       </visual>
+      <!-- vo motor NEMA17 o dau canh tay 2, chia xuong -->
+      <visual>
+        <origin xyz="${link2_len} 0 ${-wrist_motor/2}" rpy="0 0 0"/>
+        <geometry><box size="${wrist_motor} ${wrist_motor} ${wrist_motor}"/></geometry>
+        <material name="arm_dark"/>
+      </visual>
       <xacro:arm_box_inertia m="0.2" x="${link2_len}" y="${link_thick}" z="${link_thick}"/>
     </link>
@@ -89,25 +102,59 @@
       <limit lower="${-pi}" upper="${pi}" effort="10.0" velocity="2.0"/>
     </joint>
+    <!-- ===== J_wrist: cum trang xoay 360 do duoi motor (continuous) ===== -->
+    <link name="arm_wrist">
+      <visual>
+        <origin xyz="0 0 ${-wrist_len/2}" rpy="0 0 0"/>
+        <geometry><cylinder radius="0.045" length="${wrist_len}"/></geometry>
+        <material name="arm_white"/>
+      </visual>
+      <xacro:arm_box_inertia m="0.15" x="0.09" y="0.09" z="${wrist_len}"/>
+    </link>
+    <joint name="J_wrist" type="continuous">
+      <parent link="arm_link2"/>
+      <child link="arm_wrist"/>
+      <origin xyz="${link2_len} 0 ${-wrist_motor}" rpy="0 0 0"/>
+      <axis xyz="0 0 1"/>
+    </joint>
+    <!-- ===== De gripper (gan duoi cum co tay xoay) ===== -->
     <link name="arm_gripper_base">
       <visual>
         <origin xyz="0 0 0" rpy="0 0 0"/>
-        <geometry><box size="0.04 ${grip_open} 0.03"/></geometry>
+        <geometry><box size="0.04 ${grip_open} 0.025"/></geometry>
         <material name="arm_white"/>
       </visual>
-      <xacro:arm_box_inertia m="0.1" x="0.04" y="${grip_open}" z="0.03"/>
+      <xacro:arm_box_inertia m="0.1" x="0.04" y="${grip_open}" z="0.025"/>
     </link>
     <joint name="J_grip_mount" type="fixed">
-      <parent link="arm_link2"/>
+      <parent link="arm_wrist"/>
       <child link="arm_gripper_base"/>
-      <origin xyz="${link2_len} 0 0" rpy="0 0 0"/>
+      <origin xyz="0 0 ${-wrist_len}" rpy="0 0 0"/>
     </joint>
-    <link name="arm_finger_left">
-      <visual>
-        <origin xyz="${finger_len/2} 0 0" rpy="0 0 0"/>
-        <geometry><box size="${finger_len} ${finger_thick} 0.03"/></geometry>
-        <material name="arm_white"/>
-      </visual>
-      <xacro:arm_box_inertia m="0.03" x="${finger_len}" y="${finger_thick}" z="0.03"/>
-    </link>
+    <!-- ===== 2 ngam CONG om vat tron (prismatic doi xung theo truc Y) =====
+         Moi ngam la 1 cung tron (xap xi bang torus -> dung box cong gia:
+         RViz khong co arc primitive nen dung 3 box ghep thanh cung). -->
+    <xacro:macro name="curved_finger" params="name side">
+      <link name="${name}">
+        <!-- 3 doan box ghep thanh cung om -->
+        <visual>
+          <origin xyz="${finger_r} 0 ${-0.03}" rpy="0 0 0"/>
+          <geometry><box size="0.02 ${finger_thick} 0.06"/></geometry>
+          <material name="arm_white"/>
+        </visual>
+        <visual>
+          <origin xyz="${finger_r*0.7} ${side*finger_r*0.7} ${-0.03}" rpy="0 0 ${side*0.8}"/>
+          <geometry><box size="0.02 ${finger_thick} 0.06"/></geometry>
+          <material name="arm_white"/>
+        </visual>
+        <visual>
+          <origin xyz="${finger_r*0.2} ${side*finger_r} ${-0.03}" rpy="0 0 ${side*1.4}"/>
+          <geometry><box size="0.02 ${finger_thick} 0.06"/></geometry>
+          <material name="arm_white"/>
+        </visual>
+        <xacro:arm_box_inertia m="0.03" x="0.06" y="0.06" z="0.06"/>
+      </link>
+    </xacro:macro>
+    <xacro:curved_finger name="arm_finger_left"  side="1"/>
+    <xacro:curved_finger name="arm_finger_right" side="-1"/>
     <joint name="J_grip" type="prismatic">
       <parent link="arm_gripper_base"/>
@@ -117,12 +164,4 @@
       <limit lower="0.0" upper="${grip_open/2}" effort="20.0" velocity="0.1"/>
     </joint>
-    <link name="arm_finger_right">
-      <visual>
-        <origin xyz="${finger_len/2} 0 0" rpy="0 0 0"/>
-        <geometry><box size="${finger_len} ${finger_thick} 0.03"/></geometry>
-        <material name="arm_white"/>
-      </visual>
-      <xacro:arm_box_inertia m="0.03" x="${finger_len}" y="${finger_thick}" z="0.03"/>
-    </link>
     <joint name="J_grip_mirror" type="prismatic">
       <parent link="arm_gripper_base"/>

Commit message: Add Gazebo simulation support for arm
Integrate Gazebo-based simulation for the SCARA arm: add ros2_control xacro, top-level sim xacro, Gazebo world, controller config, and a launch to spawn the robot and load controllers. Update CMakeLists to install config and worlds, and package.xml to add runtime dependencies (gazebo_ros, gazebo_ros2_control, controller_manager, joint_state_broadcaster, joint_trajectory_controller). Modify arm.xacro to add collision geometry and simplify gripper fingers for reliable collision/grasping in Gazebo. README updated with usage and example commands to build, launch, and command the arm.

File: ros2_ws/src/arm_description/urdf/arm.xacro (robot description, xacro)
@@ -6,4 +6,5 @@
      + gripper kep 2 ngam cong om vat (mo/khep).
      Don vi: met, kg, rad. Macro doc lap, parent gan tuy y.
+     Co them <collision> de Gazebo tinh va cham / kep duoc vat.
      ========================================================================= -->
 <robot xmlns:xacro="http://www.ros.org/wiki/xacro" name="scara_arm">
@@ -15,10 +16,8 @@
   <xacro:property name="z_travel"     value="0.40"/>
   <xacro:property name="arm_mass"     value="0.5"/>
-  <!-- co tay = motor NEMA17 chia xuong + cum trang xoay theo -->
-  <xacro:property name="wrist_motor"  value="0.042"/>  <!-- NEMA17 ~42mm -->
-  <xacro:property name="wrist_len"    value="0.07"/>   <!-- cao cum co tay (motor+de) -->
-  <!-- gripper: 2 ngam cong om vat tron -->
-  <xacro:property name="grip_open"    value="0.20"/>   <!-- mo toi da ~20cm -->
-  <xacro:property name="finger_r"     value="0.05"/>   <!-- ban kinh cung ngam -->
+  <xacro:property name="wrist_motor"  value="0.042"/>
+  <xacro:property name="wrist_len"    value="0.07"/>
+  <xacro:property name="grip_open"    value="0.20"/>
+  <xacro:property name="finger_r"     value="0.05"/>
   <xacro:property name="finger_thick" value="0.015"/>
   <xacro:macro name="arm_box_inertia" params="m x y z">
@@ -57,4 +56,8 @@
         <material name="arm_blue"/>
       </visual>
+      <collision>
+        <origin xyz="0 0 0" rpy="0 0 0"/>
+        <geometry><box size="0.06 0.06 0.05"/></geometry>
+      </collision>
       <xacro:arm_box_inertia m="0.2" x="0.06" y="0.06" z="0.05"/>
     </link>
@@ -72,4 +75,8 @@
         <material name="arm_blue"/>
       </visual>
+      <collision>
+        <origin xyz="${link1_len/2} 0 0" rpy="0 0 0"/>
+        <geometry><box size="${link1_len} ${link_thick} ${link_thick}"/></geometry>
+      </collision>
       <xacro:arm_box_inertia m="0.3" x="${link1_len}" y="${link_thick}" z="${link_thick}"/>
     </link>
@@ -87,5 +94,4 @@
         <material name="arm_blue"/>
       </visual>
-      <!-- vo motor NEMA17 o dau canh tay 2, chia xuong -->
       <visual>
         <origin xyz="${link2_len} 0 ${-wrist_motor/2}" rpy="0 0 0"/>
@@ -93,4 +99,8 @@
         <material name="arm_dark"/>
       </visual>
+      <collision>
+        <origin xyz="${link2_len/2} 0 0" rpy="0 0 0"/>
+        <geometry><box size="${link2_len} ${link_thick} ${link_thick}"/></geometry>
+      </collision>
       <xacro:arm_box_inertia m="0.2" x="${link2_len}" y="${link_thick}" z="${link_thick}"/>
     </link>
@@ -102,5 +112,4 @@
       <limit lower="${-pi}" upper="${pi}" effort="10.0" velocity="2.0"/>
     </joint>
-    <!-- ===== J_wrist: cum trang xoay 360 do duoi motor (continuous) ===== -->
     <link name="arm_wrist">
       <visual>
@@ -109,4 +118,8 @@
         <material name="arm_white"/>
       </visual>
+      <collision>
+        <origin xyz="0 0 ${-wrist_len/2}" rpy="0 0 0"/>
+        <geometry><cylinder radius="0.045" length="${wrist_len}"/></geometry>
+      </collision>
       <xacro:arm_box_inertia m="0.15" x="0.09" y="0.09" z="${wrist_len}"/>
     </link>
@@ -117,5 +130,4 @@
       <axis xyz="0 0 1"/>
     </joint>
-    <!-- ===== De gripper (gan duoi cum co tay xoay) ===== -->
     <link name="arm_gripper_base">
       <visual>
@@ -124,4 +136,8 @@
         <material name="arm_white"/>
       </visual>
+      <collision>
+        <origin xyz="0 0 0" rpy="0 0 0"/>
+        <geometry><box size="0.04 ${grip_open} 0.025"/></geometry>
+      </collision>
       <xacro:arm_box_inertia m="0.1" x="0.04" y="${grip_open}" z="0.025"/>
     </link>
@@ -131,34 +147,25 @@
       <origin xyz="0 0 ${-wrist_len}" rpy="0 0 0"/>
     </joint>
-    <!-- ===== 2 ngam CONG om vat tron (prismatic doi xung theo truc Y) =====
-         Moi ngam la 1 cung tron (xap xi bang torus -> dung box cong gia:
-         RViz khong co arc primitive nen dung 3 box ghep thanh cung). -->
-    <xacro:macro name="curved_finger" params="name side">
+    <!-- 2 ngam: dung box don gian co COLLISION de kep duoc vat trong Gazebo -->
+    <xacro:macro name="grip_finger" params="name">
       <link name="${name}">
-        <!-- 3 doan box ghep thanh cung om -->
         <visual>
-          <origin xyz="${finger_r} 0 ${-0.03}" rpy="0 0 0"/>
-          <geometry><box size="0.02 ${finger_thick} 0.06"/></geometry>
+          <origin xyz="${finger_r} 0 -0.03" rpy="0 0 0"/>
+          <geometry><box size="${finger_r*2} ${finger_thick} 0.06"/></geometry>
           <material name="arm_white"/>
         </visual>
-        <visual>
-          <origin xyz="${finger_r*0.7} ${side*finger_r*0.7} ${-0.03}" rpy="0 0 ${side*0.8}"/>
-          <geometry><box size="0.02 ${finger_thick} 0.06"/></geometry>
-          <material name="arm_white"/>
-        </visual>
-        <visual>
-          <origin xyz="${finger_r*0.2} ${side*finger_r} ${-0.03}" rpy="0 0 ${side*1.4}"/>
-          <geometry><box size="0.02 ${finger_thick} 0.06"/></geometry>
-          <material name="arm_white"/>
-        </visual>
-        <xacro:arm_box_inertia m="0.03" x="0.06" y="0.06" z="0.06"/>
+        <collision>
+          <origin xyz="${finger_r} 0 -0.03" rpy="0 0 0"/>
+          <geometry><box size="${finger_r*2} ${finger_thick} 0.06"/></geometry>
+        </collision>
+        <xacro:arm_box_inertia m="0.03" x="${finger_r*2}" y="${finger_thick}" z="0.06"/>
       </link>
     </xacro:macro>
-    <xacro:curved_finger name="arm_finger_left"  side="1"/>
-    <xacro:curved_finger name="arm_finger_right" side="-1"/>
+    <xacro:grip_finger name="arm_finger_left"/>
+    <xacro:grip_finger name="arm_finger_right"/>
     <joint name="J_grip" type="prismatic">
       <parent link="arm_gripper_base"/>
       <child link="arm_finger_left"/>
-      <origin xyz="0 0 0" rpy="0 0 0"/>
+      <origin xyz="0 ${finger_thick} 0" rpy="0 0 0"/>
       <axis xyz="0 1 0"/>
       <limit lower="0.0" upper="${grip_open/2}" effort="20.0" velocity="0.1"/>
@@ -167,5 +174,5 @@
       <parent link="arm_gripper_base"/>
       <child link="arm_finger_right"/>
-      <origin xyz="0 0 0" rpy="0 0 0"/>
+      <origin xyz="0 ${-finger_thick} 0" rpy="0 0 0"/>
       <axis xyz="0 -1 0"/>
       <mimic joint="J_grip" multiplier="1.0" offset="0.0"/>
