Commit message: Add orbbec_bringup package; tweak Gazebo launch
Add a new ROS2 package 'orbbec_bringup' (launch files, config, package metadata, setup, resource and README) to publish the static TF and integrate an Orbbec Astra Pro driver. Update ros2_ws/.gitignore to allow local vendor checkouts and add third_party/README.md. Modify robot_description/launch/gazebo.launch.py to add 'gui' and 'load_controllers' launch args and conditionally spawn controllers. Minor URDF cleanup (removed duplicated mesh/collision block) and update STM32 language.settings env-hash.

File: ros2_ws/src/robot_description/urdf/robot.urdf.xacro (robot description, xacro)
@@ -33,9 +33,4 @@
       </geometry>
       <material name="grey"/>
-    </visual>
-    <collision>
-      <origin xyz="-1.674842 -0.764810 -1.092814" rpy="${cad_to_ros_rpy}"/>
-      <geometry>
-        <mesh filename="package://robot_description/meshes/chassis.stl"
               scale="${mesh_scale} ${mesh_scale} ${mesh_scale}"/>
       </geometry>

Commit message: Add chassis collision mesh to URDF
Introduce a <collision> element to ros2_ws/src/robot_description/urdf/robot.urdf.xacro for the chassis using package://robot_description/meshes/chassis.stl with mesh_scale and rpy set to ${cad_to_ros_rpy}. The change includes the specified origin (xyz="-1.674842 -0.764810 -1.092814") and also closes the visual block. This provides proper collision geometry for simulation and planning.

File: ros2_ws/src/robot_description/urdf/robot.urdf.xacro (robot description, xacro)
@@ -33,4 +33,9 @@
       </geometry>
       <material name="grey"/>
+    </visual>
+    <collision>
+      <origin xyz="-1.674842 -0.764810 -1.092814" rpy="${cad_to_ros_rpy}"/>
+      <geometry>
+        <mesh filename="package://robot_description/meshes/chassis.stl"
               scale="${mesh_scale} ${mesh_scale} ${mesh_scale}"/>
       </geometry>
