Commit message: Document ROS2 workspace and update robot model

File: ros2_ws/src/robot_description/urdf/common_properties.xacro (robot description, xacro)
@@ -7,34 +7,37 @@
 <robot xmlns:xacro="http://www.ros.org/wiki/xacro">
   <!-- ===== THAN XE (base / chassis) ===== -->
-  <!-- Kich thuoc that: Dai 0.74 x Rong 0.55 x Cao 0.34 (m) -->
-  <xacro:property name="base_length" value="0.74"/>   <!-- truc X (toi/lui) -->
+  <!-- Do tu chassis.stl: Dai 0.730 x Rong 0.550 x Cao 0.305 (m). -->
+  <xacro:property name="base_length" value="0.73"/>   <!-- truc X (toi/lui) -->
   <xacro:property name="base_width"  value="0.55"/>   <!-- truc Y (trai/phai) -->
-  <xacro:property name="base_height" value="0.34"/>   <!-- truc Z (cao) -->
+  <xacro:property name="base_height" value="0.305"/>  <!-- truc Z (cao) -->
   <xacro:property name="base_mass"   value="40.0"/>   <!-- UOC LUONG: doi theo can that -->
-  <!-- Co thanh nhom dinh hinh (extrusion). Mac dinh 2020 = 0.02m.
-       Do lai thanh that roi doi dung 1 so nay (vd 4040 -> 0.04). -->
-  <xacro:property name="profile_size" value="0.02"/>
+  <!-- ===== CAD mesh transform ===== -->
+  <!-- STL dung mm va truc CAD: X=trai/phai, Y=cao, Z=truoc/sau.
+       ROS: X=truoc, Y=trai, Z=cao. -->
+  <xacro:property name="mesh_scale" value="0.001"/>
+  <xacro:property name="cad_to_ros_rpy" value="1.57079632679 0 1.57079632679"/>
   <!-- ===== BANH CHINH (driven wheels) ===== -->
-  <!-- Banh do tren-xuong 0.20m => duong kinh 0.20 => ban kinh 0.10 -->
-  <xacro:property name="wheel_radius" value="0.10"/>
+  <!-- Do tu drive-wheel STL: duong kinh xap xi 0.1945m, day 0.050m. -->
+  <xacro:property name="wheel_radius" value="0.09725"/>
   <xacro:property name="wheel_width"  value="0.05"/>
   <xacro:property name="wheel_mass"   value="2.0"/>
-  <!-- Khoang cach giua 2 banh chinh (track / wheel separation), tam-toi-tam.
-       separation = base_width + wheel_width = 0.55 + 0.05 = 0.60.
-       RAT QUAN TRONG cho odometry/diff_drive. -->
-  <xacro:property name="wheel_separation" value="${base_width + wheel_width}"/>
-  <!-- Banh chinh nam GIUA than theo truc X (diff-drive co dien) -->
+  <!-- Khoang cach tam-tam do truc CAD: 981.06 - 548.56 = 432.50mm. -->
+  <xacro:property name="wheel_separation" value="0.4325"/>
+  <!-- Vi tri tam banh so voi tam base_link, lay tu CAD. -->
   <xacro:property name="wheel_xoff" value="0.0"/>
-  <!-- ===== BANH PHU (caster, xoay tu do) ===== -->
-  <!-- Dung bi cau (sphere): don gian, khong motor, lan moi huong. -->
-  <xacro:property name="caster_radius" value="0.05"/>
+  <xacro:property name="wheel_zoff" value="-0.10753"/>
+  <!-- ===== BANH PHU ===== -->
+  <!-- Kich thuoc STL phu khoang 0.169 x 0.171m. -->
+  <xacro:property name="caster_radius" value="0.0855"/>
   <xacro:property name="caster_mass"   value="0.5"/>
-  <xacro:property name="caster_xoff" value="${base_length/2 - 0.08}"/>
-  <xacro:property name="caster_yoff" value="${base_width/2 - 0.08}"/>
+  <!-- Vi tri 4 banh phu do tu tam mesh, giu dung CAD. -->
+  <xacro:property name="caster_front_x" value="0.2900"/>
+  <xacro:property name="caster_rear_x"  value="-0.2900"/>
+  <xacro:property name="caster_left_y"  value="0.15225"/>
+  <xacro:property name="caster_right_y" value="-0.12275"/>
+  <xacro:property name="caster_zoff" value="-0.118005"/>
   <!-- ===== CHIEU CAO LAP DAT ===== -->
-  <!-- Day banh chinh cham dat (z=0). Tam truc banh o z = wheel_radius.
-       Tam bi caster o z = caster_radius. -->
-  <xacro:property name="base_z" value="${wheel_radius + base_height/2}"/>
-  <xacro:property name="caster_zoff" value="${-(base_height/2 + (wheel_radius - caster_radius))}"/>
+  <!-- Base_link la tam khung. Dat theo day banh chinh trong CAD. -->
+  <xacro:property name="base_z" value="0.20478"/>
   <!-- ===== INERTIA MACROS ===== -->
   <!-- Khoi hop dac -->

File: ros2_ws/src/robot_description/urdf/robot.urdf.xacro (robot description, xacro)
@@ -2,5 +2,5 @@
 <!-- =========================================================================
      robot.urdf.xacro  FILE CHINH (top-level)
-     AMR differential-drive: 2 banh chinh co motor + 4 caster bi cau tu do.
+     AMR differential-drive: 2 banh chinh co motor + 4 banh phu tu do.
      Cay frame chuan Nav2:
        base_footprint -> base_link -> (wheels, casters, lidar, imu)
@@ -13,5 +13,4 @@
   <xacro:include filename="$(find robot_description)/urdf/common_properties.xacro"/>
   <xacro:include filename="$(find robot_description)/urdf/materials.xacro"/>
-  <xacro:include filename="$(find robot_description)/urdf/chassis_frame.xacro"/>
   <xacro:include filename="$(find robot_description)/urdf/wheels.xacro"/>
   <xacro:include filename="$(find robot_description)/urdf/sensors.xacro"/>
@@ -26,11 +25,18 @@
   <!-- ===== base_link (than xe) ===== -->
   <link name="base_link">
-    <!-- VISUAL = khung nhom ho (nhieu thanh box), nhin giong xe that -->
-    <xacro:chassis_frame L="${base_length}" W="${base_width}" H="${base_height}" p="${profile_size}"/>
-    <!-- COLLISION = 1 khoi hop bao ngoai (don gian, nhe, an toan cho Nav2). -->
+    <!-- Mesh goc tu CAD; scale mm -> m va doi truc CAD -> ROS. -->
+    <visual>
+      <origin xyz="-1.674842 -0.764810 -1.092814" rpy="${cad_to_ros_rpy}"/>
+      <geometry>
+        <mesh filename="package://robot_description/meshes/chassis.stl"
+              scale="${mesh_scale} ${mesh_scale} ${mesh_scale}"/>
+      </geometry>
+      <material name="grey"/>
+    </visual>
     <collision>
-      <origin xyz="0 0 0" rpy="0 0 0"/>
+      <origin xyz="-1.674842 -0.764810 -1.092814" rpy="${cad_to_ros_rpy}"/>
       <geometry>
-        <box size="${base_length} ${base_width} ${base_height}"/>
+        <mesh filename="package://robot_description/meshes/chassis.stl"
+              scale="${mesh_scale} ${mesh_scale} ${mesh_scale}"/>
       </geometry>
     </collision>
@@ -41,11 +47,23 @@
   </gazebo>
   <!-- ===== Banh chinh ===== -->
-  <xacro:drive_wheel prefix="left"  reflect="1"/>
-  <xacro:drive_wheel prefix="right" reflect="-1"/>
-  <!-- ===== 4 caster o 4 goc ===== -->
-  <xacro:caster_wheel prefix="front_left"  xpos="1"  ypos="1"/>
-  <xacro:caster_wheel prefix="front_right" xpos="1"  ypos="-1"/>
-  <xacro:caster_wheel prefix="rear_left"   xpos="-1" ypos="1"/>
-  <xacro:caster_wheel prefix="rear_right"  xpos="-1" ypos="-1"/>
+  <xacro:drive_wheel prefix="left"  reflect="1"
+                     mesh_file="left_drive_wheel.stl"
+                     mesh_x="-1.674844" mesh_y="-0.981060" mesh_z="-0.985314"/>
+  <xacro:drive_wheel prefix="right" reflect="-1"
+                     mesh_file="right_drive_wheel.stl"
+                     mesh_x="-1.674844" mesh_y="-0.548560" mesh_z="-0.985314"/>
+  <!-- ===== 4 banh phu o 4 goc ===== -->
+  <xacro:caster_wheel prefix="front_left" xpos="${caster_front_x}" ypos="${caster_left_y}"
+                       mesh_file="front_left_caster.stl"
+                       mesh_x="-1.964838" mesh_y="-0.917062" mesh_z="-0.974809"/>
+  <xacro:caster_wheel prefix="front_right" xpos="${caster_front_x}" ypos="${caster_right_y}"
+                       mesh_file="front_right_caster.stl"
+                       mesh_x="-1.964857" mesh_y="-0.642145" mesh_z="-0.974809"/>
+  <xacro:caster_wheel prefix="rear_left" xpos="${caster_rear_x}" ypos="${caster_left_y}"
+                       mesh_file="rear_left_caster.stl"
+                       mesh_x="-1.384831" mesh_y="-0.917062" mesh_z="-0.974809"/>
+  <xacro:caster_wheel prefix="rear_right" xpos="${caster_rear_x}" ypos="${caster_right_y}"
+                       mesh_file="rear_right_caster.stl"
+                       mesh_x="-1.384831" mesh_y="-0.642062" mesh_z="-0.974809"/>
   <!-- ===== ros2_control ===== -->
   <xacro:robot_ros2_control use_sim="$(arg use_sim)"/>

File: ros2_ws/src/robot_description/urdf/robot_expanded_hw.urdf (robot description, URDF)
Before this commit: robot amr_robot, 10 links, 9 joints
Links:
- link base_link: geometry collision mesh filename=package://robot_description/meshes/chassis.stl scale=0.001 0.001 0.001; visual mesh filename=package://robot_description/meshes/chassis.stl scale=0.001 0.001 0.001
- link front_left_caster_link: geometry collision mesh filename=package://robot_description/meshes/front_left_caster.stl scale=0.001 0.001 0.001; visual mesh filename=package://robot_description/meshes/front_left_caster.stl scale=0.001 0.001 0.001
- link front_right_caster_link: geometry collision mesh filename=package://robot_description/meshes/front_right_caster.stl scale=0.001 0.001 0.001; visual mesh filename=package://robot_description/meshes/front_right_caster.stl scale=0.001 0.001 0.001
- link left_wheel_link: geometry collision mesh filename=package://robot_description/meshes/left_drive_wheel.stl scale=0.001 0.001 0.001; visual mesh filename=package://robot_description/meshes/left_drive_wheel.stl scale=0.001 0.001 0.001
- link rear_left_caster_link: geometry collision mesh filename=package://robot_description/meshes/rear_left_caster.stl scale=0.001 0.001 0.001; visual mesh filename=package://robot_description/meshes/rear_left_caster.stl scale=0.001 0.001 0.001
- link rear_right_caster_link: geometry collision mesh filename=package://robot_description/meshes/rear_right_caster.stl scale=0.001 0.001 0.001; visual mesh filename=package://robot_description/meshes/rear_right_caster.stl scale=0.001 0.001 0.001
- link right_wheel_link: geometry collision mesh filename=package://robot_description/meshes/right_drive_wheel.stl scale=0.001 0.001 0.001; visual mesh filename=package://robot_description/meshes/right_drive_wheel.stl scale=0.001 0.001 0.001
Joints:
- joint base_joint: origin xyz=0 0 0.27 rpy=0 0 0 -> xyz=0 0 0.20478 rpy=0 0 0
- joint front_left_caster_joint: origin xyz=0.29 0.195 -0.22000000000000003 rpy=0 0 0 -> xyz=0.29 0.15225 -0.118005 rpy=0 0 0
- joint front_right_caster_joint: origin xyz=0.29 -0.195 -0.22000000000000003 rpy=0 0 0 -> xyz=0.29 -0.12275 -0.118005 rpy=0 0 0
- joint left_wheel_joint: origin xyz=0.0 0.30000000000000004 -0.17 rpy=0 0 0 -> xyz=0.0 0.21625 -0.10753 rpy=0 0 0
- joint lidar_joint: origin xyz=0.27 0 0.195 rpy=0 0 0 -> xyz=0.265 0 0.1775 rpy=0 0 0
- joint rear_left_caster_joint: origin xyz=-0.29 0.195 -0.22000000000000003 rpy=0 0 0 -> xyz=-0.29 0.15225 -0.118005 rpy=0 0 0
- joint rear_right_caster_joint: origin xyz=-0.29 -0.195 -0.22000000000000003 rpy=0 0 0 -> xyz=-0.29 -0.12275 -0.118005 rpy=0 0 0
- joint right_wheel_joint: origin xyz=0.0 -0.30000000000000004 -0.17 rpy=0 0 0 -> xyz=0.0 -0.21625 -0.10753 rpy=0 0 0

File: ros2_ws/src/robot_description/urdf/robot_expanded_sim.urdf (robot description, URDF)
Before this commit: robot amr_robot, 10 links, 9 joints
Links:
- link base_link: geometry collision mesh filename=package://robot_description/meshes/chassis.stl scale=0.001 0.001 0.001; visual mesh filename=package://robot_description/meshes/chassis.stl scale=0.001 0.001 0.001
- link front_left_caster_link: geometry collision mesh filename=package://robot_description/meshes/front_left_caster.stl scale=0.001 0.001 0.001; visual mesh filename=package://robot_description/meshes/front_left_caster.stl scale=0.001 0.001 0.001
- link front_right_caster_link: geometry collision mesh filename=package://robot_description/meshes/front_right_caster.stl scale=0.001 0.001 0.001; visual mesh filename=package://robot_description/meshes/front_right_caster.stl scale=0.001 0.001 0.001
- link left_wheel_link: geometry collision mesh filename=package://robot_description/meshes/left_drive_wheel.stl scale=0.001 0.001 0.001; visual mesh filename=package://robot_description/meshes/left_drive_wheel.stl scale=0.001 0.001 0.001
- link rear_left_caster_link: geometry collision mesh filename=package://robot_description/meshes/rear_left_caster.stl scale=0.001 0.001 0.001; visual mesh filename=package://robot_description/meshes/rear_left_caster.stl scale=0.001 0.001 0.001
- link rear_right_caster_link: geometry collision mesh filename=package://robot_description/meshes/rear_right_caster.stl scale=0.001 0.001 0.001; visual mesh filename=package://robot_description/meshes/rear_right_caster.stl scale=0.001 0.001 0.001
- link right_wheel_link: geometry collision mesh filename=package://robot_description/meshes/right_drive_wheel.stl scale=0.001 0.001 0.001; visual mesh filename=package://robot_description/meshes/right_drive_wheel.stl scale=0.001 0.001 0.001
Joints:
- joint base_joint: origin xyz=0 0 0.27 rpy=0 0 0 -> xyz=0 0 0.20478 rpy=0 0 0
- joint front_left_caster_joint: origin xyz=0.29 0.195 -0.22000000000000003 rpy=0 0 0 -> xyz=0.29 0.15225 -0.118005 rpy=0 0 0
- joint front_right_caster_joint: origin xyz=0.29 -0.195 -0.22000000000000003 rpy=0 0 0 -> xyz=0.29 -0.12275 -0.118005 rpy=0 0 0
- joint left_wheel_joint: origin xyz=0.0 0.30000000000000004 -0.17 rpy=0 0 0 -> xyz=0.0 0.21625 -0.10753 rpy=0 0 0
- joint lidar_joint: origin xyz=0.27 0 0.195 rpy=0 0 0 -> xyz=0.265 0 0.1775 rpy=0 0 0
- joint rear_left_caster_joint: origin xyz=-0.29 0.195 -0.22000000000000003 rpy=0 0 0 -> xyz=-0.29 0.15225 -0.118005 rpy=0 0 0
- joint rear_right_caster_joint: origin xyz=-0.29 -0.195 -0.22000000000000003 rpy=0 0 0 -> xyz=-0.29 -0.12275 -0.118005 rpy=0 0 0
- joint right_wheel_joint: origin xyz=0.0 -0.30000000000000004 -0.17 rpy=0 0 0 -> xyz=0.0 -0.21625 -0.10753 rpy=0 0 0

File: ros2_ws/src/robot_description/urdf/wheels.xacro (robot description, xacro)
@@ -2,24 +2,24 @@
 <!-- =========================================================================
      wheels.xacro
-     Macro cho bánh chính (driven, continuous joint) và caster (bi cầu, fixed
-     vì bi lăn tự do trong sim — không cần joint quay riêng cho bi cầu).
+     Macro cho bánh chính (driven, continuous joint) và 4 bánh phụ.
      ========================================================================= -->
 <robot xmlns:xacro="http://www.ros.org/wiki/xacro">
   <!-- ===== BÁNH CHÍNH (có motor) ===== -->
   <!-- prefix: left/right ; reflect: +1 (trái) / -1 (phải) -->
-  <xacro:macro name="drive_wheel" params="prefix reflect">
+  <xacro:macro name="drive_wheel" params="prefix reflect mesh_file mesh_x mesh_y mesh_z">
     <link name="${prefix}_wheel_link">
       <visual>
-        <!-- cylinder mặc định trục theo Z; xoay 90° quanh X để trục về Y -->
-        <origin xyz="0 0 0" rpy="${pi/2} 0 0"/>
+        <origin xyz="${mesh_x} ${mesh_y} ${mesh_z}" rpy="${cad_to_ros_rpy}"/>
         <geometry>
-          <cylinder radius="${wheel_radius}" length="${wheel_width}"/>
+          <mesh filename="package://robot_description/meshes/${mesh_file}"
+                scale="${mesh_scale} ${mesh_scale} ${mesh_scale}"/>
         </geometry>
         <material name="black"/>
       </visual>
       <collision>
-        <origin xyz="0 0 0" rpy="${pi/2} 0 0"/>
+        <origin xyz="${mesh_x} ${mesh_y} ${mesh_z}" rpy="${cad_to_ros_rpy}"/>
         <geometry>
-          <cylinder radius="${wheel_radius}" length="${wheel_width}"/>
+          <mesh filename="package://robot_description/meshes/${mesh_file}"
+                scale="${mesh_scale} ${mesh_scale} ${mesh_scale}"/>
         </geometry>
       </collision>
@@ -31,6 +31,6 @@
       <parent link="base_link"/>
       <child  link="${prefix}_wheel_link"/>
-      <!-- đặt bánh sát hông: y = +/- wheel_separation/2 ; z = xuống tới tâm trục -->
-      <origin xyz="${wheel_xoff} ${reflect * wheel_separation/2} ${-base_height/2}"
+      <!-- Vi tri tam banh lay tu CAD -->
+      <origin xyz="${wheel_xoff} ${reflect * wheel_separation/2} ${wheel_zoff}"
               rpy="0 0 0"/>
       <axis xyz="0 1 0"/>
@@ -47,24 +47,32 @@
     </gazebo>
   </xacro:macro>
-  <!-- ===== CASTER (bi cầu, tự do) ===== -->
-  <!-- prefix: vd front_left ; xpos/ypos: dấu của offset X/Y -->
-  <xacro:macro name="caster_wheel" params="prefix xpos ypos">
+  <!-- ===== BANH PHU ===== -->
+  <!-- Hinh dang lay tu STL; co cau swivel chua duoc mo phong. -->
+  <xacro:macro name="caster_wheel" params="prefix xpos ypos mesh_file mesh_x mesh_y mesh_z">
     <link name="${prefix}_caster_link">
       <visual>
-        <geometry><sphere radius="${caster_radius}"/></geometry>
-        <material name="dark_grey"/>
+        <origin xyz="${mesh_x} ${mesh_y} ${mesh_z}" rpy="${cad_to_ros_rpy}"/>
+        <geometry>
+          <mesh filename="package://robot_description/meshes/${mesh_file}"
+                scale="${mesh_scale} ${mesh_scale} ${mesh_scale}"/>
+        </geometry>
+        <material name="black"/>
       </visual>
       <collision>
-        <geometry><sphere radius="${caster_radius}"/></geometry>
+        <origin xyz="${mesh_x} ${mesh_y} ${mesh_z}" rpy="${cad_to_ros_rpy}"/>
+        <geometry>
+          <mesh filename="package://robot_description/meshes/${mesh_file}"
+                scale="${mesh_scale} ${mesh_scale} ${mesh_scale}"/>
+        </geometry>
       </collision>
       <xacro:sphere_inertia m="${caster_mass}" r="${caster_radius}"/>
     </link>
-    <!-- fixed joint: bi cầu lăn tự do nhờ ma sát thấp (mu≈0), không cần motor/joint quay -->
+    <!-- fixed joint: chi mo phong hinh dang va tiep xuc, chua co swivel joint -->
     <joint name="${prefix}_caster_joint" type="fixed">
       <parent link="base_link"/>
       <child  link="${prefix}_caster_link"/>
-      <origin xyz="${xpos * caster_xoff} ${ypos * caster_yoff} ${caster_zoff}" rpy="0 0 0"/>
+      <origin xyz="${xpos} ${ypos} ${caster_zoff}" rpy="0 0 0"/>
     </joint>
-    <!-- ma sát ~0 để bi trượt/lăn mọi hướng như caster thật -->
+    <!-- Ma sat thap de banh phu khong keo le robot qua nhieu. -->
     <gazebo reference="${prefix}_caster_link">
       <mu1>0.0</mu1>

Commit message: Improve Gazebo compatibility and physics
This commit updates the Gazebo launch flow to set the plugin path and optionally disable ros2_control generation via a new `use_ros2_control` argument. It strips XML comments before URDF processing to avoid xacro parsing issues, keeps the robot spawn height stable, and adds a cleaner launch setup using `OpaqueFunction`.

It also simplifies collision geometry by replacing heavy STL meshes with lightweight box, cylinder, and sphere collisions to improve Gazebo/ODE performance. The caster z-offset is adjusted so the support wheels contact the ground correctly without tipping the robot.

File: ros2_ws/src/robot_description/urdf/common_properties.xacro (robot description, xacro)
@@ -36,5 +36,7 @@
   <xacro:property name="caster_left_y"  value="0.15225"/>
   <xacro:property name="caster_right_y" value="-0.12275"/>
-  <xacro:property name="caster_zoff" value="-0.118005"/>
+  <!-- Ha xuong de banh phu CHAM DAT (day = day banh chinh) -> robot dung vung,
+       khong lat. caster_zoff = caster_radius - base_z = 0.0855 - 0.20478. -->
+  <xacro:property name="caster_zoff" value="-0.11928"/>
   <!-- ===== CHIEU CAO LAP DAT ===== -->
   <!-- Base_link la tam khung. Dat theo day banh chinh trong CAD. -->

File: ros2_ws/src/robot_description/urdf/robot.urdf.xacro (robot description, xacro)
@@ -10,4 +10,5 @@
   <!-- true = chay Gazebo ; false = hardware that -->
   <xacro:arg name="use_sim" default="true"/>
+  <xacro:arg name="use_ros2_control" default="true"/>
   <!-- ===== Include cac phan ===== -->
   <xacro:include filename="$(find robot_description)/urdf/common_properties.xacro"/>
@@ -34,9 +35,10 @@
       <material name="grey"/>
     </visual>
+    <!-- Collision = box don gian (khong dung mesh) de Gazebo/ODE dung va cham
+         NHANH. Mesh chi tiet lam physics cham vai phut trong VM. -->
     <collision>
-      <origin xyz="-1.674842 -0.764810 -1.092814" rpy="${cad_to_ros_rpy}"/>
+      <origin xyz="0 0 0" rpy="0 0 0"/>
       <geometry>
-        <mesh filename="package://robot_description/meshes/chassis.stl"
-              scale="${mesh_scale} ${mesh_scale} ${mesh_scale}"/>
+        <box size="${base_length} ${base_width} ${base_height}"/>
       </geometry>
     </collision>
@@ -67,4 +69,6 @@
                        mesh_x="-1.384831" mesh_y="-0.642062" mesh_z="-0.974809"/>
   <!-- ===== ros2_control ===== -->
-  <xacro:robot_ros2_control use_sim="$(arg use_sim)"/>
+  <xacro:if value="$(arg use_ros2_control)">
+    <xacro:robot_ros2_control use_sim="$(arg use_sim)"/>
+  </xacro:if>
 </robot>

File: ros2_ws/src/robot_description/urdf/wheels.xacro (robot description, xacro)
@@ -17,9 +17,9 @@
         <material name="black"/>
       </visual>
+      <!-- Collision = cylinder (truc quay quanh Y). Nhanh hon mesh nhieu. -->
       <collision>
-        <origin xyz="${mesh_x} ${mesh_y} ${mesh_z}" rpy="${cad_to_ros_rpy}"/>
+        <origin xyz="0 0 0" rpy="1.5707963 0 0"/>
         <geometry>
-          <mesh filename="package://robot_description/meshes/${mesh_file}"
-                scale="${mesh_scale} ${mesh_scale} ${mesh_scale}"/>
+          <cylinder radius="${wheel_radius}" length="${wheel_width}"/>
         </geometry>
       </collision>
@@ -59,9 +59,9 @@
         <material name="black"/>
       </visual>
+      <!-- Collision = sphere don gian thay cho mesh phu. -->
       <collision>
-        <origin xyz="${mesh_x} ${mesh_y} ${mesh_z}" rpy="${cad_to_ros_rpy}"/>
+        <origin xyz="0 0 0" rpy="0 0 0"/>
         <geometry>
-          <mesh filename="package://robot_description/meshes/${mesh_file}"
-                scale="${mesh_scale} ${mesh_scale} ${mesh_scale}"/>
+          <sphere radius="${caster_radius}"/>
         </geometry>
       </collision>
