Commit message: .

File: ros2_ws/src/robot_description/urdf/materials.xacro (robot description, xacro)
@@ -7,4 +7,6 @@
   <material name="black">  <color rgba="0.05 0.05 0.05 1.0"/></material>
   <material name="blue">   <color rgba="0.1 0.3 0.8 1.0"/></material>
+  <material name="green">  <color rgba="0.1 0.8 0.2 1.0"/></material>
+  <material name="yellow"> <color rgba="0.9 0.8 0.1 1.0"/></material>
   <material name="white">  <color rgba="0.9 0.9 0.9 1.0"/></material>
 </robot>

File: ros2_ws/src/robot_description/urdf/robot.urdf.xacro (robot description, xacro)
@@ -4,5 +4,5 @@
      AMR differential-drive: 2 banh chinh co motor + 4 banh phu tu do.
      Cay frame chuan Nav2:
-       base_footprint -> base_link -> (wheels, casters, lidar, imu)
+       base_footprint -> base_link -> (wheels, casters, lidar, sonar1/2, imu)
      Build: xacro robot.urdf.xacro use_sim:=true > robot.urdf
      ========================================================================= -->

File: ros2_ws/src/robot_description/urdf/sensors.xacro (robot description, xacro)
@@ -2,13 +2,13 @@
 <!-- =========================================================================
      sensors.xacro
-     LiDAR 2D + IMU — cần cho SLAM / Nav2.
+     LiDAR 2D + IMU + 2 SR04T.
      Vị trí gắn là ƯỚC LƯỢNG: chỉnh lại theo chỗ bạn lắp cảm biến thật.
      ========================================================================= -->
 <robot xmlns:xacro="http://www.ros.org/wiki/xacro">
   <!-- ============================ LiDAR 2D ============================ -->
-  <!-- Gắn trên nóc, phía trước, giữa theo Y -->
+  <!-- LiDAR gắn giữa nóc xe theo vị trí lắp thực tế. -->
   <xacro:property name="lidar_radius" value="0.04"/>
   <xacro:property name="lidar_height" value="0.05"/>
-  <xacro:property name="lidar_x" value="${base_length/2 - 0.10}"/>
+  <xacro:property name="lidar_x" value="0.0"/>
   <xacro:property name="lidar_z" value="${base_height/2 + lidar_height/2}"/>
   <link name="lidar_link">
@@ -64,4 +64,35 @@
     </sensor>
   </gazebo>
+  <!-- =========================== SR04T pair =========================== -->
+  <!-- Range frames point along local +X. SONAR1 looks forward; SONAR2 is
+       rotated pi radians to look backward. Positions are temporary until
+       measured on the finished chassis. -->
+  <xacro:property name="sonar_body_depth" value="0.025"/>
+  <xacro:property name="sonar_body_width" value="0.045"/>
+  <xacro:property name="sonar_body_height" value="0.025"/>
+  <xacro:property name="sonar_mount_z" value="0.0"/>
+  <xacro:macro name="sr04t_link" params="name x yaw material">
+    <link name="${name}">
+      <visual>
+        <!-- Link origin is the acoustic face; body extends into the chassis. -->
+        <origin xyz="${-sonar_body_depth/2} 0 0" rpy="0 0 0"/>
+        <geometry>
+          <box size="${sonar_body_depth} ${sonar_body_width} ${sonar_body_height}"/>
+        </geometry>
+        <material name="${material}"/>
+      </visual>
+    </link>
+    <joint name="${name}_joint" type="fixed">
+      <parent link="base_link"/>
+      <child link="${name}"/>
+      <origin xyz="${x} 0 ${sonar_mount_z}" rpy="0 0 ${yaw}"/>
+    </joint>
+  </xacro:macro>
+  <!-- Schematic SONAR1 (PB0/PB1): front centre, facing +X. -->
+  <xacro:sr04t_link name="sonar1_link"
+                     x="${base_length/2}" yaw="0" material="green"/>
+  <!-- Schematic SONAR2 (PB11/PB12): rear centre, facing -X. -->
+  <xacro:sr04t_link name="sonar2_link"
+                     x="${-base_length/2}" yaw="3.14159265359" material="yellow"/>
   <!-- ============================== IMU =============================== -->
   <link name="imu_link">
