Commit message: Add CAD body meshes, xacro updates & tests
Add 35 STL CAD meshes and integrate them into the robot xacro/URDF (28 body meshes). Update urdf common properties (body_mesh_origin, base box dims/collision), add xacro macro body_visual, and switch heavy mesh collisions to simple primitives (box/cylinder/sphere) for faster simulation. Add LiDAR mesh and two sonar links, adjust sensor origins/inertia, and tweak caster/wheel positions. Add a Python unit test (test_mesh_references.py) and enable it from CMakeLists when BUILD_TESTING is on. Update README and expanded URDFs accordingly. Co-authored-by: Copilot <223556219+Copilot@users.noreply.github.com>

File: robot/ros2_ws/src/robot_description/urdf/common_properties.xacro (robot description, xacro)
@@ -7,8 +7,8 @@
 <robot xmlns:xacro="http://www.ros.org/wiki/xacro">
   <!-- ===== THAN XE (base / chassis) ===== -->
-  <!-- Do tu chassis.stl: Dai 0.730 x Rong 0.550 x Cao 0.305 (m). -->
-  <xacro:property name="base_length" value="0.73"/>   <!-- truc X (toi/lui) -->
-  <xacro:property name="base_width"  value="0.55"/>   <!-- truc Y (trai/phai) -->
-  <xacro:property name="base_height" value="0.305"/>  <!-- truc Z (cao) -->
+  <!-- Bao ngoai cua toan bo 28 mesh than xe, khong tinh banh va LiDAR (m). -->
+  <xacro:property name="base_length" value="0.805422607"/>  <!-- truc X (toi/lui) -->
+  <xacro:property name="base_width"  value="0.566226318"/>  <!-- truc Y (trai/phai) -->
+  <xacro:property name="base_height" value="0.416"/>        <!-- truc Z (cao) -->
   <xacro:property name="base_mass"   value="40.0"/>   <!-- UOC LUONG: doi theo can that -->
   <!-- ===== CAD mesh transform ===== -->
@@ -17,4 +17,21 @@
   <xacro:property name="mesh_scale" value="0.001"/>
   <xacro:property name="cad_to_ros_rpy" value="1.57079632679 0 1.57079632679"/>
+  <!-- Moi body STL duoc export trong cung toa do assembly. Origin nay dat
+       tam khung CAD tai base_link; khong can offset rieng cho tung part. -->
+  <xacro:property name="body_mesh_origin" value="-1.674842 -0.764810 -1.092814"/>
+  <!-- Tam box bao ngoai lech khoi tam khung vi vo xe khong doi xung. -->
+  <xacro:property name="base_collision_x" value="-0.001387776"/>
+  <xacro:property name="base_collision_y" value="0.001886533"/>
+  <xacro:property name="base_collision_z" value="0.055499721"/>
+  <xacro:macro name="body_visual" params="mesh_file material:=grey">
+    <visual>
+      <origin xyz="${body_mesh_origin}" rpy="${cad_to_ros_rpy}"/>
+      <geometry>
+        <mesh filename="package://robot_description/meshes/${mesh_file}"
+              scale="${mesh_scale} ${mesh_scale} ${mesh_scale}"/>
+      </geometry>
+      <material name="${material}"/>
+    </visual>
+  </xacro:macro>
   <!-- ===== BANH CHINH (driven wheels) ===== -->
   <!-- Do tu drive-wheel STL: duong kinh xap xi 0.1945m, day 0.050m. -->

File: robot/ros2_ws/src/robot_description/urdf/robot.urdf.xacro (robot description, xacro)
@@ -26,17 +26,38 @@
   <!-- ===== base_link (than xe) ===== -->
   <link name="base_link">
-    <!-- Mesh goc tu CAD; scale mm -> m va doi truc CAD -> ROS. -->
-    <visual>
-      <origin xyz="-1.674842 -0.764810 -1.092814" rpy="${cad_to_ros_rpy}"/>
-      <geometry>
-        <mesh filename="package://robot_description/meshes/chassis.stl"
-              scale="${mesh_scale} ${mesh_scale} ${mesh_scale}"/>
-      </geometry>
-      <material name="grey"/>
-    </visual>
+    <!-- Cac mesh duoc export theo toa do assembly, scale mm -> m. -->
+    <xacro:body_visual mesh_file="chassis.stl" material="dark_grey"/>
+    <xacro:body_visual mesh_file="lower_center_1.stl"/>
+    <xacro:body_visual mesh_file="lower_center_2.stl"/>
+    <xacro:body_visual mesh_file="upper_corner_1_6.stl"/>
+    <xacro:body_visual mesh_file="upper_corner_1_7.stl"/>
+    <xacro:body_visual mesh_file="upper_corner_2_1.stl"/>
+    <xacro:body_visual mesh_file="upper_corner_2_2.stl"/>
+    <xacro:body_visual mesh_file="lower_corner_1_1.stl"/>
+    <xacro:body_visual mesh_file="lower_corner_1_2.stl"/>
+    <xacro:body_visual mesh_file="lower_corner_2_1.stl"/>
+    <xacro:body_visual mesh_file="lower_corner_2_2.stl"/>
+    <xacro:body_visual mesh_file="top_cover.stl"/>
+    <xacro:body_visual mesh_file="lower_plate_1_1.stl"/>
+    <xacro:body_visual mesh_file="lower_plate_1_2.stl"/>
+    <xacro:body_visual mesh_file="lower_plate_3_1.stl"/>
+    <xacro:body_visual mesh_file="lower_plate_3_2.stl"/>
+    <xacro:body_visual mesh_file="lower_shell_1.stl"/>
+    <xacro:body_visual mesh_file="lower_shell_2.stl"/>
+    <xacro:body_visual mesh_file="body_shell_1_1.stl"/>
+    <xacro:body_visual mesh_file="body_shell_1_2.stl"/>
+    <xacro:body_visual mesh_file="body_shell_l_middle_1_1.stl"/>
+    <xacro:body_visual mesh_file="body_shell_l_middle_1.stl"/>
+    <xacro:body_visual mesh_file="body_shell_l_1.stl"/>
+    <xacro:body_visual mesh_file="body_shell_l_2.stl"/>
+    <xacro:body_visual mesh_file="body_end_shell_1.stl"/>
+    <xacro:body_visual mesh_file="body_end_shell_2.stl"/>
+    <xacro:body_visual mesh_file="spacer_5.stl"/>
+    <xacro:body_visual mesh_file="spacer_7.stl"/>
     <!-- Collision = box don gian (khong dung mesh) de Gazebo/ODE dung va cham
          NHANH. Mesh chi tiet lam physics cham vai phut trong VM. -->
     <collision>
-      <origin xyz="0 0 0" rpy="0 0 0"/>
+      <origin xyz="${base_collision_x} ${base_collision_y} ${base_collision_z}"
+              rpy="0 0 0"/>
       <geometry>
         <box size="${base_length} ${base_width} ${base_height}"/>

File: robot/ros2_ws/src/robot_description/urdf/robot_expanded_hw.urdf (robot description, URDF)
Before this commit: robot amr_robot, 10 links, 9 joints
Links:
- added link sonar1_link; visual box size=0.025 0.045 0.025
- added link sonar2_link; visual box size=0.025 0.045 0.025
- link base_link: geometry collision box size=0.805422607 0.566226318 0.416; visual mesh filename=package://robot_description/meshes/body_end_shell_1.stl scale=0.001 0.001 0.001
- link front_left_caster_link: geometry collision sphere radius=0.0855; visual mesh filename=package://robot_description/meshes/front_left_caster.stl scale=0.001 0.001 0.001
- link front_right_caster_link: geometry collision sphere radius=0.0855; visual mesh filename=package://robot_description/meshes/front_right_caster.stl scale=0.001 0.001 0.001
- link left_wheel_link: geometry collision cylinder length=0.05 radius=0.09725; visual mesh filename=package://robot_description/meshes/left_drive_wheel.stl scale=0.001 0.001 0.001
- link lidar_link: geometry collision cylinder length=0.0405 radius=0.038679688; visual mesh filename=package://robot_description/meshes/lidar_body.stl scale=0.001 0.001 0.001
- link rear_left_caster_link: geometry collision sphere radius=0.0855; visual mesh filename=package://robot_description/meshes/rear_left_caster.stl scale=0.001 0.001 0.001
- link rear_right_caster_link: geometry collision sphere radius=0.0855; visual mesh filename=package://robot_description/meshes/rear_right_caster.stl scale=0.001 0.001 0.001
- link right_wheel_link: geometry collision cylinder length=0.05 radius=0.09725; visual mesh filename=package://robot_description/meshes/right_drive_wheel.stl scale=0.001 0.001 0.001
Joints:
- added joint sonar1_link_joint: type fixed, parent base_link, child sonar1_link, origin xyz=0.4013235275 0 0.0 rpy=0 0 0
- added joint sonar2_link_joint: type fixed, parent base_link, child sonar2_link, origin xyz=-0.4040990795 0 0.0 rpy=0 0 3.14159265359
- joint front_left_caster_joint: origin xyz=0.29 0.15225 -0.118005 rpy=0 0 0 -> xyz=0.29 0.15225 -0.11928 rpy=0 0 0
- joint front_right_caster_joint: origin xyz=0.29 -0.12275 -0.118005 rpy=0 0 0 -> xyz=0.29 -0.12275 -0.11928 rpy=0 0 0
- joint lidar_joint: origin xyz=0.265 0 0.1775 rpy=0 0 0 -> xyz=-0.004433431 0.003998868 0.283749721 rpy=0 0 0
- joint rear_left_caster_joint: origin xyz=-0.29 0.15225 -0.118005 rpy=0 0 0 -> xyz=-0.29 0.15225 -0.11928 rpy=0 0 0
- joint rear_right_caster_joint: origin xyz=-0.29 -0.12275 -0.118005 rpy=0 0 0 -> xyz=-0.29 -0.12275 -0.11928 rpy=0 0 0

File: robot/ros2_ws/src/robot_description/urdf/robot_expanded_sim.urdf (robot description, URDF)
Before this commit: robot amr_robot, 10 links, 9 joints
Links:
- added link sonar1_link; visual box size=0.025 0.045 0.025
- added link sonar2_link; visual box size=0.025 0.045 0.025
- link base_link: geometry collision box size=0.805422607 0.566226318 0.416; visual mesh filename=package://robot_description/meshes/body_end_shell_1.stl scale=0.001 0.001 0.001
- link front_left_caster_link: geometry collision sphere radius=0.0855; visual mesh filename=package://robot_description/meshes/front_left_caster.stl scale=0.001 0.001 0.001
- link front_right_caster_link: geometry collision sphere radius=0.0855; visual mesh filename=package://robot_description/meshes/front_right_caster.stl scale=0.001 0.001 0.001
- link left_wheel_link: geometry collision cylinder length=0.05 radius=0.09725; visual mesh filename=package://robot_description/meshes/left_drive_wheel.stl scale=0.001 0.001 0.001
- link lidar_link: geometry collision cylinder length=0.0405 radius=0.038679688; visual mesh filename=package://robot_description/meshes/lidar_body.stl scale=0.001 0.001 0.001
- link rear_left_caster_link: geometry collision sphere radius=0.0855; visual mesh filename=package://robot_description/meshes/rear_left_caster.stl scale=0.001 0.001 0.001
- link rear_right_caster_link: geometry collision sphere radius=0.0855; visual mesh filename=package://robot_description/meshes/rear_right_caster.stl scale=0.001 0.001 0.001
- link right_wheel_link: geometry collision cylinder length=0.05 radius=0.09725; visual mesh filename=package://robot_description/meshes/right_drive_wheel.stl scale=0.001 0.001 0.001
Joints:
- added joint sonar1_link_joint: type fixed, parent base_link, child sonar1_link, origin xyz=0.4013235275 0 0.0 rpy=0 0 0
- added joint sonar2_link_joint: type fixed, parent base_link, child sonar2_link, origin xyz=-0.4040990795 0 0.0 rpy=0 0 3.14159265359
- joint front_left_caster_joint: origin xyz=0.29 0.15225 -0.118005 rpy=0 0 0 -> xyz=0.29 0.15225 -0.11928 rpy=0 0 0
- joint front_right_caster_joint: origin xyz=0.29 -0.12275 -0.118005 rpy=0 0 0 -> xyz=0.29 -0.12275 -0.11928 rpy=0 0 0
- joint lidar_joint: origin xyz=0.265 0 0.1775 rpy=0 0 0 -> xyz=-0.004433431 0.003998868 0.283749721 rpy=0 0 0
- joint rear_left_caster_joint: origin xyz=-0.29 0.15225 -0.118005 rpy=0 0 0 -> xyz=-0.29 0.15225 -0.11928 rpy=0 0 0
- joint rear_right_caster_joint: origin xyz=-0.29 -0.12275 -0.118005 rpy=0 0 0 -> xyz=-0.29 -0.12275 -0.11928 rpy=0 0 0

File: robot/ros2_ws/src/robot_description/urdf/sensors.xacro (robot description, xacro)
@@ -3,17 +3,23 @@
      sensors.xacro
      LiDAR 2D + IMU + 2 SR04T.
-     Vị trí gắn là ƯỚC LƯỢNG: chỉnh lại theo chỗ bạn lắp cảm biến thật.
+     LiDAR lấy từ CAD; vị trí sonar và IMU vẫn là ƯỚC LƯỢNG.
      ========================================================================= -->
 <robot xmlns:xacro="http://www.ros.org/wiki/xacro">
   <!-- ============================ LiDAR 2D ============================ -->
-  <!-- LiDAR gắn giữa nóc xe theo vị trí lắp thực tế. -->
-  <xacro:property name="lidar_radius" value="0.04"/>
-  <xacro:property name="lidar_height" value="0.05"/>
-  <xacro:property name="lidar_x" value="0.0"/>
-  <xacro:property name="lidar_z" value="${base_height/2 + lidar_height/2}"/>
+  <!-- Kich thuoc, tam va mesh origin do truc tiep tu lidar_body.stl. -->
+  <xacro:property name="lidar_radius" value="0.038679688"/>
+  <xacro:property name="lidar_height" value="0.0405"/>
+  <xacro:property name="lidar_x" value="-0.004433431"/>
+  <xacro:property name="lidar_y" value="0.003998868"/>
+  <xacro:property name="lidar_z" value="0.283749721"/>
   <link name="lidar_link">
     <visual>
-      <geometry><cylinder radius="${lidar_radius}" length="${lidar_height}"/></geometry>
-      <material name="blue"/>
+      <origin xyz="-1.670408569 -0.768808868 -1.376563721"
+              rpy="${cad_to_ros_rpy}"/>
+      <geometry>
+        <mesh filename="package://robot_description/meshes/lidar_body.stl"
+              scale="${mesh_scale} ${mesh_scale} ${mesh_scale}"/>
+      </geometry>
+      <material name="black"/>
     </visual>
     <collision>
@@ -25,5 +31,5 @@
     <parent link="base_link"/>
     <child  link="lidar_link"/>
-    <origin xyz="${lidar_x} 0 ${lidar_z}" rpy="0 0 0"/>
+    <origin xyz="${lidar_x} ${lidar_y} ${lidar_z}" rpy="0 0 0"/>
   </joint>
   <gazebo reference="lidar_link">
@@ -91,8 +97,8 @@
   <!-- Schematic SONAR1 (PB0/PB1): front centre, facing +X. -->
   <xacro:sr04t_link name="sonar1_link"
-                     x="${base_length/2}" yaw="0" material="green"/>
+                     x="${base_collision_x + base_length/2}" yaw="0" material="green"/>
   <!-- Schematic SONAR2 (PB11/PB12): rear centre, facing -X. -->
   <xacro:sr04t_link name="sonar2_link"
-                     x="${-base_length/2}" yaw="3.14159265359" material="yellow"/>
+                     x="${base_collision_x - base_length/2}" yaw="3.14159265359" material="yellow"/>
   <!-- ============================== IMU =============================== -->
   <link name="imu_link">
