Commit message: Align robot CAD with real geometry and dev setup
Update the robot URDF, wheel/mesh dimensions, and odometry defaults to match the current CAD and real hardware (0.4325 m wheelbase, 0.09725 m radius, base_footprint TF). Add the Ubuntu VMware dev Docker Compose flow and a mesh-reference regression test to guard the CAD assembly and mesh origins.

File: robot/ros2_ws/src/robot_description/urdf/common_properties.xacro (robot description, xacro)
@@ -7,8 +7,8 @@
 <robot xmlns:xacro="http://www.ros.org/wiki/xacro">
   <!-- ===== THAN XE (base / chassis) ===== -->
-  <!-- Bao ngoai cua toan bo 28 mesh than xe, khong tinh banh va LiDAR (m). -->
-  <xacro:property name="base_length" value="0.805422607"/>  <!-- truc X (toi/lui) -->
-  <xacro:property name="base_width"  value="0.566226318"/>  <!-- truc Y (trai/phai) -->
-  <xacro:property name="base_height" value="0.416"/>        <!-- truc Z (cao) -->
+  <!-- Bao ngoai 28 mesh than xe, khong tinh banh, LiDAR va camera (m). -->
+  <xacro:property name="base_length" value="0.802199951"/>  <!-- truc X (toi/lui) -->
+  <xacro:property name="base_width"  value="0.562799988"/>  <!-- truc Y (trai/phai) -->
+  <xacro:property name="base_height" value="0.421100037"/>  <!-- truc Z (cao) -->
   <xacro:property name="base_mass"   value="40.0"/>   <!-- UOC LUONG: doi theo can that -->
   <!-- ===== CAD mesh transform ===== -->
@@ -19,10 +19,21 @@
   <!-- Moi body STL duoc export trong cung toa do assembly. Origin nay dat
        tam khung CAD tai base_link; khong can offset rieng cho tung part. -->
-  <xacro:property name="body_mesh_origin" value="-1.674842 -0.764810 -1.092814"/>
+  <xacro:property name="body_mesh_origin" value="-1.638492310 -0.744854355 -1.164497711"/>
   <!-- Tam box bao ngoai lech khoi tam khung vi vo xe khong doi xung. -->
-  <xacro:property name="base_collision_x" value="-0.001387776"/>
-  <xacro:property name="base_collision_y" value="0.001886533"/>
-  <xacro:property name="base_collision_z" value="0.055499721"/>
+  <xacro:property name="base_collision_x" value="0.0"/>
+  <xacro:property name="base_collision_y" value="0.000049973"/>
+  <xacro:property name="base_collision_z" value="0.056"/>
   <xacro:macro name="body_visual" params="mesh_file material:=grey">
+    <visual>
+      <origin xyz="${body_mesh_origin}" rpy="${cad_to_ros_rpy}"/>
+      <geometry>
+        <mesh filename="package://robot_description/meshes/${mesh_file}"
+              scale="${mesh_scale} ${mesh_scale} ${mesh_scale}"/>
+      </geometry>
+      <material name="${material}"/>
+    </visual>
+  </xacro:macro>
+  <!-- Phu kien giu toa do assembly nhung khong tham gia tinh body envelope. -->
+  <xacro:macro name="assembly_visual" params="mesh_file material:=grey">
     <visual>
       <origin xyz="${body_mesh_origin}" rpy="${cad_to_ros_rpy}"/>
@@ -43,5 +54,5 @@
   <!-- Vi tri tam banh so voi tam base_link, lay tu CAD. -->
   <xacro:property name="wheel_xoff" value="0.0"/>
-  <xacro:property name="wheel_zoff" value="-0.10753"/>
+  <xacro:property name="wheel_zoff" value="-0.10955"/>
   <!-- ===== BANH PHU ===== -->
   <!-- Kich thuoc STL phu khoang 0.169 x 0.171m. -->
@@ -54,9 +65,9 @@
   <xacro:property name="caster_right_y" value="-0.12275"/>
   <!-- Ha xuong de banh phu CHAM DAT (day = day banh chinh) -> robot dung vung,
-       khong lat. caster_zoff = caster_radius - base_z = 0.0855 - 0.20478. -->
-  <xacro:property name="caster_zoff" value="-0.11928"/>
+       khong lat. caster_zoff = caster_radius - base_z = 0.0855 - 0.2068. -->
+  <xacro:property name="caster_zoff" value="-0.1213"/>
   <!-- ===== CHIEU CAO LAP DAT ===== -->
   <!-- Base_link la tam khung. Dat theo day banh chinh trong CAD. -->
-  <xacro:property name="base_z" value="0.20478"/>
+  <xacro:property name="base_z" value="0.2068"/>
   <!-- ===== INERTIA MACROS ===== -->
   <!-- Khoi hop dac -->

File: robot/ros2_ws/src/robot_description/urdf/robot.urdf.xacro (robot description, xacro)
@@ -55,4 +55,8 @@
     <xacro:body_visual mesh_file="spacer_5.stl"/>
     <xacro:body_visual mesh_file="spacer_7.stl"/>
+    <!-- Camera va ga camera chi la visual. camera_link van do
+         orbbec_bringup publish de tranh hai nguon TF trung nhau. -->
+    <xacro:assembly_visual mesh_file="camera_mount.stl" material="dark_grey"/>
+    <xacro:assembly_visual mesh_file="camera_body.stl" material="black"/>
     <!-- Collision = box don gian (khong dung mesh) de Gazebo/ODE dung va cham
          NHANH. Mesh chi tiet lam physics cham vai phut trong VM. -->
@@ -72,21 +76,21 @@
   <xacro:drive_wheel prefix="left"  reflect="1"
                      mesh_file="left_drive_wheel.stl"
-                     mesh_x="-1.674844" mesh_y="-0.981060" mesh_z="-0.985314"/>
+                     mesh_x="-1.638492371" mesh_y="-0.961104370" mesh_z="-1.054947693"/>
   <xacro:drive_wheel prefix="right" reflect="-1"
                      mesh_file="right_drive_wheel.stl"
-                     mesh_x="-1.674844" mesh_y="-0.548560" mesh_z="-0.985314"/>
+                     mesh_x="-1.638492371" mesh_y="-0.528604355" mesh_z="-1.054947723"/>
   <!-- ===== 4 banh phu o 4 goc ===== -->
   <xacro:caster_wheel prefix="front_left" xpos="${caster_front_x}" ypos="${caster_left_y}"
                        mesh_file="front_left_caster.stl"
-                       mesh_x="-1.964838" mesh_y="-0.917062" mesh_z="-0.974809"/>
+                       mesh_x="-1.928486755" mesh_y="-0.897107056" mesh_z="-1.044442749"/>
   <xacro:caster_wheel prefix="front_right" xpos="${caster_front_x}" ypos="${caster_right_y}"
                        mesh_file="front_right_caster.stl"
-                       mesh_x="-1.964857" mesh_y="-0.642145" mesh_z="-0.974809"/>
+                       mesh_x="-1.928504944" mesh_y="-0.622189758" mesh_z="-1.044442749"/>
   <xacro:caster_wheel prefix="rear_left" xpos="${caster_rear_x}" ypos="${caster_left_y}"
                        mesh_file="rear_left_caster.stl"
-                       mesh_x="-1.384831" mesh_y="-0.917062" mesh_z="-0.974809"/>
+                       mesh_x="-1.348479675" mesh_y="-0.897107056" mesh_z="-1.044442749"/>
   <xacro:caster_wheel prefix="rear_right" xpos="${caster_rear_x}" ypos="${caster_right_y}"
                        mesh_file="rear_right_caster.stl"
-                       mesh_x="-1.384831" mesh_y="-0.642062" mesh_z="-0.974809"/>
+                       mesh_x="-1.348479675" mesh_y="-0.622107056" mesh_z="-1.044442749"/>
   <!-- ===== ros2_control ===== -->
   <xacro:if value="$(arg use_ros2_control)">

File: robot/ros2_ws/src/robot_description/urdf/robot_expanded_hw.urdf (robot description, URDF)
Before this commit: robot amr_robot, 14 links, 13 joints
Links:
- link base_link: geometry collision box size=0.802199951 0.562799988 0.421100037; visual mesh filename=package://robot_description/meshes/body_end_shell_1.stl scale=0.001 0.001 0.001
- link lidar_link: geometry collision cylinder length=0.0405 radius=0.038679932; visual mesh filename=package://robot_description/meshes/lidar_body.stl scale=0.001 0.001 0.001
Joints:
- joint base_joint: origin xyz=0 0 0.20478 rpy=0 0 0 -> xyz=0 0 0.2068 rpy=0 0 0
- joint front_left_caster_joint: origin xyz=0.29 0.15225 -0.11928 rpy=0 0 0 -> xyz=0.29 0.15225 -0.1213 rpy=0 0 0
- joint front_right_caster_joint: origin xyz=0.29 -0.12275 -0.11928 rpy=0 0 0 -> xyz=0.29 -0.12275 -0.1213 rpy=0 0 0
- joint left_wheel_joint: origin xyz=0.0 0.21625 -0.10753 rpy=0 0 0 -> xyz=0.0 0.21625 -0.10955 rpy=0 0 0
- joint lidar_joint: origin xyz=-0.004433431 0.003998868 0.283749721 rpy=0 0 0 -> xyz=-0.001439453 0.0 0.266499969 rpy=0 0 0
- joint rear_left_caster_joint: origin xyz=-0.29 0.15225 -0.11928 rpy=0 0 0 -> xyz=-0.29 0.15225 -0.1213 rpy=0 0 0
- joint rear_right_caster_joint: origin xyz=-0.29 -0.12275 -0.11928 rpy=0 0 0 -> xyz=-0.29 -0.12275 -0.1213 rpy=0 0 0
- joint right_wheel_joint: origin xyz=0.0 -0.21625 -0.10753 rpy=0 0 0 -> xyz=0.0 -0.21625 -0.10955 rpy=0 0 0

File: robot/ros2_ws/src/robot_description/urdf/robot_expanded_sim.urdf (robot description, URDF)
Before this commit: robot amr_robot, 14 links, 13 joints
Links:
- link base_link: geometry collision box size=0.802199951 0.562799988 0.421100037; visual mesh filename=package://robot_description/meshes/body_end_shell_1.stl scale=0.001 0.001 0.001
- link lidar_link: geometry collision cylinder length=0.0405 radius=0.038679932; visual mesh filename=package://robot_description/meshes/lidar_body.stl scale=0.001 0.001 0.001
Joints:
- joint base_joint: origin xyz=0 0 0.20478 rpy=0 0 0 -> xyz=0 0 0.2068 rpy=0 0 0
- joint front_left_caster_joint: origin xyz=0.29 0.15225 -0.11928 rpy=0 0 0 -> xyz=0.29 0.15225 -0.1213 rpy=0 0 0
- joint front_right_caster_joint: origin xyz=0.29 -0.12275 -0.11928 rpy=0 0 0 -> xyz=0.29 -0.12275 -0.1213 rpy=0 0 0
- joint left_wheel_joint: origin xyz=0.0 0.21625 -0.10753 rpy=0 0 0 -> xyz=0.0 0.21625 -0.10955 rpy=0 0 0
- joint lidar_joint: origin xyz=-0.004433431 0.003998868 0.283749721 rpy=0 0 0 -> xyz=-0.001439453 0.0 0.266499969 rpy=0 0 0
- joint rear_left_caster_joint: origin xyz=-0.29 0.15225 -0.11928 rpy=0 0 0 -> xyz=-0.29 0.15225 -0.1213 rpy=0 0 0
- joint rear_right_caster_joint: origin xyz=-0.29 -0.12275 -0.11928 rpy=0 0 0 -> xyz=-0.29 -0.12275 -0.1213 rpy=0 0 0
- joint right_wheel_joint: origin xyz=0.0 -0.21625 -0.10753 rpy=0 0 0 -> xyz=0.0 -0.21625 -0.10955 rpy=0 0 0

File: robot/ros2_ws/src/robot_description/urdf/sensors.xacro (robot description, xacro)
@@ -8,12 +8,12 @@
   <!-- ============================ LiDAR 2D ============================ -->
   <!-- Kich thuoc, tam va mesh origin do truc tiep tu lidar_body.stl. -->
-  <xacro:property name="lidar_radius" value="0.038679688"/>
+  <xacro:property name="lidar_radius" value="0.038679932"/>
   <xacro:property name="lidar_height" value="0.0405"/>
-  <xacro:property name="lidar_x" value="-0.004433431"/>
-  <xacro:property name="lidar_y" value="0.003998868"/>
-  <xacro:property name="lidar_z" value="0.283749721"/>
+  <xacro:property name="lidar_x" value="-0.001439453"/>
+  <xacro:property name="lidar_y" value="0.0"/>
+  <xacro:property name="lidar_z" value="0.266499969"/>
   <link name="lidar_link">
     <visual>
-      <origin xyz="-1.670408569 -0.768808868 -1.376563721"
+      <origin xyz="-1.637052856 -0.744854340 -1.430997681"
               rpy="${cad_to_ros_rpy}"/>
       <geometry>
