Commit message: Add support for four SR04T sonars
Extend firmware, bridge and robot description to handle 4 SR04T ultrasonic sensors.

- Firmware (Core/Inc, Core/Src, .ioc): add PB13/PB14/PB15/PA6 pin defs, EXTI9_5 handler, GPIO init for TRIG/ECHO, and SR04T driver updated to SR04T_SENSOR_COUNT=4 with correct TRIG/ECHO ports/pins and round-robin scheduling. USB feedback format extended to include sonar3/sonar4 values.
- stm32_bridge: launch, node and README updated to declare/publish four sonar topics and parse the new 16-field FB format while remaining backward-compatible with the old 12-field format. Added unit test for 16-field parsing and adjusted existing test expectations.
- robot_description: URDF/xacro, READMEs and nav2 docs updated to place four sonars in the robot model and enable Nav2 RangeSensorLayer configuration examples for four sensors.
- Docs/PIN_MAP updated with new pins and hardware notes.

Backward compatibility: bridge still accepts older 12-field feedback; new 16-field format is preferred. Tests updated to cover both cases.

File: robot/ros2_ws/src/robot_description/urdf/robot_expanded_hw.urdf (robot description, URDF)
Before this commit: robot amr_robot, 12 links, 11 joints
Links:
- added link sonar3_link; visual box size=0.025 0.045 0.025
- added link sonar4_link; visual box size=0.025 0.045 0.025
Joints:
- added joint sonar3_link_joint: type fixed, parent base_link, child sonar3_link, origin xyz=-0.4040990795 0.284999692 0.0 rpy=0 0 2.35619449019
- added joint sonar4_link_joint: type fixed, parent base_link, child sonar4_link, origin xyz=-0.4040990795 -0.281226626 0.0 rpy=0 0 -2.35619449019
- joint sonar1_link_joint: origin xyz=0.4013235275 0 0.0 rpy=0 0 0 -> xyz=0.4013235275 0.284999692 0.0 rpy=0 0 0.78539816340
- joint sonar2_link_joint: origin xyz=-0.4040990795 0 0.0 rpy=0 0 3.14159265359 -> xyz=0.4013235275 -0.281226626 0.0 rpy=0 0 -0.78539816340

File: robot/ros2_ws/src/robot_description/urdf/robot_expanded_sim.urdf (robot description, URDF)
Before this commit: robot amr_robot, 12 links, 11 joints
Links:
- added link sonar3_link; visual box size=0.025 0.045 0.025
- added link sonar4_link; visual box size=0.025 0.045 0.025
Joints:
- added joint sonar3_link_joint: type fixed, parent base_link, child sonar3_link, origin xyz=-0.4040990795 0.284999692 0.0 rpy=0 0 2.35619449019
- added joint sonar4_link_joint: type fixed, parent base_link, child sonar4_link, origin xyz=-0.4040990795 -0.281226626 0.0 rpy=0 0 -2.35619449019
- joint sonar1_link_joint: origin xyz=0.4013235275 0 0.0 rpy=0 0 0 -> xyz=0.4013235275 0.284999692 0.0 rpy=0 0 0.78539816340
- joint sonar2_link_joint: origin xyz=-0.4040990795 0 0.0 rpy=0 0 3.14159265359 -> xyz=0.4013235275 -0.281226626 0.0 rpy=0 0 -0.78539816340

File: robot/ros2_ws/src/robot_description/urdf/sensors.xacro (robot description, xacro)
@@ -2,5 +2,5 @@
 <!-- =========================================================================
      sensors.xacro
-     LiDAR 2D + IMU + 2 SR04T.
+     LiDAR 2D + IMU + 4 SR04T.
      LiDAR lấy từ CAD; vị trí sonar và IMU vẫn là ƯỚC LƯỢNG.
      ========================================================================= -->
@@ -70,13 +70,14 @@
     </sensor>
   </gazebo>
-  <!-- =========================== SR04T pair =========================== -->
-  <!-- Range frames point along local +X. SONAR1 looks forward; SONAR2 is
-       rotated pi radians to look backward. Positions are temporary until
-       measured on the finished chassis. -->
+  <!-- =========================== SR04T x4 =========================== -->
+  <!-- Range frames point along local +X. All four SR04T sit at the four
+       corners of the chassis, each facing diagonally outward (yaw = +-45 deg
+       from the corner's bisector). Positions are temporary until measured
+       on the finished chassis. -->
   <xacro:property name="sonar_body_depth" value="0.025"/>
   <xacro:property name="sonar_body_width" value="0.045"/>
   <xacro:property name="sonar_body_height" value="0.025"/>
   <xacro:property name="sonar_mount_z" value="0.0"/>
-  <xacro:macro name="sr04t_link" params="name x yaw material">
+  <xacro:macro name="sr04t_link" params="name x y yaw material">
     <link name="${name}">
       <visual>
@@ -92,13 +93,31 @@
       <parent link="base_link"/>
       <child link="${name}"/>
-      <origin xyz="${x} 0 ${sonar_mount_z}" rpy="0 0 ${yaw}"/>
+      <origin xyz="${x} ${y} ${sonar_mount_z}" rpy="0 0 ${yaw}"/>
     </joint>
   </xacro:macro>
-  <!-- Schematic SONAR1 (PB0/PB1): front centre, facing +X. -->
+  <!-- Schematic SONAR1 (PB0/PB1): front-left corner, facing +45 deg (out
+       to front-left diagonal). -->
   <xacro:sr04t_link name="sonar1_link"
-                     x="${base_collision_x + base_length/2}" yaw="0" material="green"/>
-  <!-- Schematic SONAR2 (PB11/PB12): rear centre, facing -X. -->
+                     x="${base_collision_x + base_length/2}"
+                     y="${base_collision_y + base_width/2}"
+                     yaw="0.78539816340" material="green"/>
+  <!-- Schematic SONAR2 (PB11/PB12): front-right corner, facing -45 deg (out
+       to front-right diagonal). -->
   <xacro:sr04t_link name="sonar2_link"
-                     x="${base_collision_x - base_length/2}" yaw="3.14159265359" material="yellow"/>
+                     x="${base_collision_x + base_length/2}"
+                     y="${base_collision_y - base_width/2}"
+                     yaw="-0.78539816340" material="yellow"/>
+  <!-- Schematic SONAR3 (PB13/PB14): rear-left corner, facing 135 deg (out
+       to rear-left diagonal). -->
+  <xacro:sr04t_link name="sonar3_link"
+                     x="${base_collision_x - base_length/2}"
+                     y="${base_collision_y + base_width/2}"
+                     yaw="2.35619449019" material="blue"/>
+  <!-- Schematic SONAR4 (PB15/PA6): rear-right corner, facing -135 deg (out
+       to rear-right diagonal). -->
+  <xacro:sr04t_link name="sonar4_link"
+                     x="${base_collision_x - base_length/2}"
+                     y="${base_collision_y - base_width/2}"
+                     yaw="-2.35619449019" material="orange"/>
   <!-- ============================== IMU =============================== -->
   <link name="imu_link">
